File: bussedBreakoutSSOP24.kicad_pcb (KiCad board)
At the start: 2 copper layers, 2.9 x 2.9 mm, 49 parts, among them J1 Conn_01x12_Pin, J10 Conn_01x06_Pin, J11 Conn_01x06_Pin, J12 Conn_01x06_Pin, J13 Conn_01x06_Pin, J14 Conn_01x06_Pin, J15 Conn_01x06_Pin, J16 Conn_01x06_Pin, J17 Conn_01x06_Pin, J18 Conn_01x06_Pin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

Commit message: Change to SSOP24 breakout
Parts:
- added J26: Conn_01x24_Pin, SMD:SMD_grid_2x12_0402, F.Cu at (33.0, 52.1)
- added J27: Conn_01x24_Pin, SMD:SMD_grid_2x12_0402, F.Cu at (33.0, 54.6)
- J21: value SOP-24 -> SSOP-24; footprint SMD:SOP-24_3.9-7.5mmx15.4mm_P1.27mm -> SMD:SSOP-24_3.9-7.5mmx8.2mm_P0.65mm
- moved J24 17.8 mm to (33.0, 34.3)
- moved J25 5.08 mm to (33.0, 49.5)
Connections:
- J12 pad 2: unconnected-(J12-Pin_2-Pad2) -> /4T
- J12 pad 5: unconnected-(J12-Pin_5-Pad5) -> /21T
- J17 pad 2: unconnected-(J17-Pin_2-Pad2) -> /9T
- J17 pad 5: unconnected-(J17-Pin_5-Pad5) -> /16T
- J20 pad 2: /12T -> unconnected-(J20-Pin_2-Pad2)
- J22 pad 15: /24T -> GND
- J22 pad 17: /24T -> GND
- J22 pad 19: /24T -> GND
- J22 pad 21: /24T -> GND
- J22 pad 23: Net-(J22-Pin_23) -> GND
- J22 pad 24: Net-(J22-Pin_23) -> unconnected-(J22-Pin_24-Pad24)
- J24 pad 10: /11T -> /4T
- J24 pad 15: /15T -> /22T
- J24 pad 16: /14T -> /21T
- J24 pad 17: /15T -> /22T
- J24 pad 18: /14T -> /21T
- J24 pad 19: /15T -> /22T
- J24 pad 20: /14T -> /21T
- J24 pad 21: /15T -> /22T
- J24 pad 22: /14T -> /21T
- J24 pad 3: /10T -> /3T
- J24 pad 4: /11T -> /4T
- J24 pad 5: /10T -> /3T
- J24 pad 6: /11T -> /4T
- J24 pad 7: /10T -> /3T
- J24 pad 8: /11T -> /4T
- J24 pad 9: /10T -> /3T
- J25 pad 10: /12T -> /10T
- J25 pad 15: /14T -> /16T
- J25 pad 16: /13T -> /15T
- J25 pad 17: /14T -> /16T
- J25 pad 18: /13T -> /15T
- J25 pad 19: /14T -> /16T
- J25 pad 20: /13T -> /15T
- J25 pad 21: /14T -> /16T
- J25 pad 22: /13T -> /15T
- J25 pad 3: /11T -> /9T
- J25 pad 4: /12T -> /10T
- J25 pad 5: /11T -> /9T
- J25 pad 6: /12T -> /10T
- J25 pad 7: /11T -> /9T
- J25 pad 8: /12T -> /10T
- J25 pad 9: /11T -> /9T
- J9 pad 5: /24T -> unconnected-(J9-Pin_5-Pad5)
Routing:
- net GND: track 52.2 -> 47.2 mm
- net VCC: track 53.3 -> 48.4 mm
- net /3T: track 2.12 -> 6.19 mm, vias 1 -> 2
- net /15T: track 2.13 -> 6.19 mm, vias 1 -> 2
- net /22T: track 2.13 -> 6.19 mm, vias 1 -> 2
- net /10T: track 2.12 -> 6.16 mm, vias 1 -> 2
- net /12: track 16.1 -> 20.0 mm
- net /1: track 15.5 -> 19.2 mm
- net /13: track 15.3 -> 18.8 mm
- net /9T: track 0.00 -> 3.45 mm, vias 0 -> 1
- net /4T: track 0.00 -> 3.45 mm, vias 0 -> 1
- net /21T: track 0.00 -> 3.45 mm, vias 0 -> 1
- net /16T: track 0.00 -> 3.45 mm, vias 0 -> 1
- net /24: track 15.7 -> 18.8 mm
- net /23: track 15.1 -> 18.0 mm
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Other:
- board text added: "0.65mm pitch"
- board text added: "SSOP-24"
- board text removed: "1.27mm pitch"
- board text removed: "SOP-24"

Commit message: Reorient power distribution jumpers to remove GND/VCC routing workaround
Parts:
- moved JP23 1.26 mm to (36.7, 57.8), turned to -135 degrees
- moved JP24 1.11 mm to (39.1, 57.7), turned to -135 degrees
- moved JP20 1.11 mm to (29.0, 57.7), turned to -135 degrees
- moved JP22 1.11 mm to (34.0, 57.7), turned to -135 degrees
- moved JP21 1.06 mm to (31.5, 57.7), turned to -135 degrees
- moved JP16 1.01 mm to (29.5, 26.2), turned to 45 degrees
- moved JP17 1.01 mm to (32.1, 26.2), turned to 45 degrees
- moved JP18 1.01 mm to (34.6, 26.2), turned to 45 degrees
- moved JP19 1.01 mm to (37.2, 26.2), turned to 45 degrees
- moved JP15 0.94 mm to (27.1, 26.3), turned to 45 degrees
Connections:
- J20 pad 2: unconnected-(J20-Pin_2-Pad2) -> /12T
- J22 pad 15: GND -> /23T
- J22 pad 16: /23T -> /24T
- J22 pad 17: GND -> /23T
- J22 pad 18: /23T -> /24T
- J22 pad 19: GND -> /23T
- J22 pad 20: /23T -> /24T
- J22 pad 21: GND -> /23T
- J22 pad 22: /23T -> /24T
- J22 pad 23: GND -> Net-(J22-Pin_23)
- J22 pad 24: unconnected-(J22-Pin_24-Pad24) -> Net-(J22-Pin_23)
- J27 pad 1: unconnected-(J27-Pin_1-Pad1) -> Net-(J27-Pin_1)
- J27 pad 10: VCC -> /12T
- J27 pad 2: VCC -> Net-(J27-Pin_1)
- J27 pad 4: VCC -> /12T
- J27 pad 6: VCC -> /12T
- J27 pad 8: VCC -> /12T
- J9 pad 5: unconnected-(J9-Pin_5-Pad5) -> /1T
Routing:
- net VCC: track 48.4 -> 52.6 mm
- net /12T: track 0.00 -> 3.45 mm, vias 0 -> 1
- net /23T: track 5.47 -> 8.21 mm
- net Net-(J27-Pin_1): track 0.00 -> 1.12 mm
- net /13T: track 2.74 -> 3.45 mm

Commit message: Fix missing T24/T23 vias
Connections:
- J22 pad 15: /23T -> /24T
- J22 pad 16: /24T -> /23T
- J22 pad 17: /23T -> /24T
- J22 pad 18: /24T -> /23T
- J22 pad 19: /23T -> /24T
- J22 pad 20: /24T -> /23T
- J22 pad 21: /23T -> /24T
- J22 pad 22: /24T -> /23T
- J9 pad 5: /1T -> /24T
Routing:
- net /24T: track 0.00 -> 3.45 mm, vias 0 -> 1
- net /23T: track 8.21 -> 5.47 mm
Changed lines of the file:
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@@
 		(fp_poly
 			(pts
-				(xy -0.15 -0.32) (xy -0.15 0.32) (xy 0.15 0.32) (xy 0.15 -0.32)
+				(xy -0.15 -0.32) (xy 0.15 -0.32) (xy 0.15 0.32) (xy -0.15 0.32)
 			)
 			(stroke
@@
 		(fp_poly
 			(pts
-				(xy -0.15 -0.32) (xy -0.15 0.32) (xy 0.15 0.32) (xy 0.15 -0.32)
+				(xy -0.15 -0.32) (xy 0.15 -0.32) (xy 0.15 0.32) (xy -0.15 0.32)
 			)
 			(stroke
@@
 		(fp_poly
 			(pts
-				(xy -0.15 -0.32) (xy -0.15 0.32) (xy 0.15 0.32) (xy 0.15 -0.32)
+				(xy -0.15 -0.32) (xy 0.15 -0.32) (xy 0.15 0.32) (xy -0.15 0.32)
 			)
 			(stroke
@@
 		(fp_poly
 			(pts
-				(xy -0.15 -0.32) (xy -0.15 0.32) (xy 0.15 0.32) (xy 0.15 -0.32)
+				(xy -0.15 -0.32) (xy 0.15 -0.32) (xy 0.15 0.32) (xy -0.15 0.32)
 			)
 			(stroke
@@
 		(fp_poly
 			(pts
-				(xy -0.15 -0.32) (xy -0.15 0.32) (xy 0.15 0.32) (xy 0.15 -0.32)
+				(xy -0.15 -0.32) (xy 0.15 -0.32) (xy 0.15 0.32) (xy -0.15 0.32)
 			)
 			(stroke
@@
 		(fp_poly
 			(pts
-				(xy -0.15 -0.32) (xy -0.15 0.32) (xy 0.15 0.32) (xy 0.15 -0.32)
+				(xy -0.15 -0.32) (xy 0.15 -0.32) (xy 0.15 0.32) (xy -0.15 0.32)
 			)
 			(stroke
@@
 		(fp_poly
 			(pts
-				(xy -0.15 -0.32) (xy -0.15 0.32) (xy 0.15 0.32) (xy 0.15 -0.32)
+				(xy -0.15 -0.32) (xy 0.15 -0.32) (xy 0.15 0.32) (xy -0.15 0.32)
 			)
 			(stroke
@@
 		(fp_poly
 			(pts
-				(xy -0.15 -0.32) (xy -0.15 0.32) (xy 0.15 0.32) (xy 0.15 -0.32)
+				(xy -0.15 -0.32) (xy 0.15 -0.32) (xy 0.15 0.32) (xy -0.15 0.32)
 			)
 			(stroke
@@
 		(fp_poly
 			(pts
-				(xy -0.15 -0.32) (xy -0.15 0.32) (xy 0.15 0.32) (xy 0.15 -0.32)
+				(xy -0.15 -0.32) (xy 0.15 -0.32) (xy 0.15 0.32) (xy -0.15 0.32)
 			)
 			(stroke
@@
 			(layers "F.Cu" "F.Mask")
 			(roundrect_rratio 0.25)
-			(net 47 "/23T")
+			(net 77 "/24T")
 			(pinfunction "Pin_15")
 			(pintype "passive")
@@
 			(layers "F.Cu" "F.Mask")
 			(roundrect_rratio 0.25)
-			(net 77 "/24T")
+			(net 47 "/23T")
 			(pinfunction "Pin_16")
 			(pintype "passive")
@@
 			(layers "F.Cu" "F.Mask")
 			(roundrect_rratio 0.25)
-			(net 47 "/23T")
+			(net 77 "/24T")
 			(pinfunction "Pin_17")
 			(pintype "passive")
@@
 			(layers "F.Cu" "F.Mask")
 			(roundrect_rratio 0.25)
-			(net 77 "/24T")
+			(net 47 "/23T")
 			(pinfunction "Pin_18")
 			(pintype "passive")
@@
 			(layers "F.Cu" "F.Mask")
 			(roundrect_rratio 0.25)
-			(net 47 "/23T")
+			(net 77 "/24T")
 			(pinfunction "Pin_19")
 			(pintype "passive")
@@
 			(layers "F.Cu" "F.Mask")
 			(roundrect_rratio 0.25)
-			(net 77 "/24T")
+			(net 47 "/23T")
 			(pinfunction "Pin_20")
 			(pintype "passive")
@@
 			(layers "F.Cu" "F.Mask")
 			(roundrect_rratio 0.25)
-			(net 47 "/23T")
+			(net 77 "/24T")
 			(pinfunction "Pin_21")
 			(pintype "passive")
@@
 			(layers "F.Cu" "F.Mask")
 			(roundrect_rratio 0.25)
-			(net 77 "/24T")
+			(net 47 "/23T")
 			(pinfunction "Pin_22")
 			(pintype "passive")
@@
 		(fp_poly
 			(pts
-				(xy -0.15 -0.32) (xy -0.15 0.32) (xy 0.15 0.32) (xy 0.15 -0.32)
+				(xy -0.15 -0.32) (xy 0.15 -0.32) (xy 0.15 0.32) (xy -0.15 0.32)
 			)
 			(stroke
@@
 			(layers "B.Cu" "B.Mask")
 			(roundrect_rratio 0.243902)
-			(net 46 "/1T")
+			(net 77 "/24T")
 			(pinfunction "Pin_5")
 			(pintype "passive")
@@
 	)
 	(gr_text "24"
-		(at 39.37 28.575 0)
+		(at 39.116 27.94 0)
 		(layer "F.SilkS")
 		(effects
@@
 	)
 	(gr_text "12"
-		(at 26.797 55.245 0)
+		(at 26.797 55.88 0)
 		(layer "F.SilkS")
 		(effects
@@
 		(net 47)
 	)
-	(segment
-		(start 34.38875 28.6487)
-		(end 37.12625 28.6487)
-		(width 0.2)
-		(layer "F.Cu")
-		(net 47)
-	)
 	(via
 		(at 35.7632 29.7688)
@@
 	)
 	(segment
+		(start 34.38875 28.6487)
+		(end 35.7632 28.6487)
+		(width 0.2)
+		(layer "F.Cu")
+		(net 77)
+	)
+	(segment
+		(start 35.7632 28.6487)
+		(end 37.12625 28.6487)
+		(width 0.2)
+		(layer "F.Cu")
+		(net 77)
+	)
+	(via
+		(at 35.7632 28.6487)
+		(size 0.6)
+		(drill 0.3)
+		(layers "F.Cu" "B.Cu")
+		(net 77)
+	)
+	(segment
+		(start 35.7575 28.643)
+		(end 35.7632 28.6487)
+		(width 0.2)
+		(layer "B.Cu")
+		(net 77)
+	)
+	(segment
+		(start 35.7575 27.94)
+		(end 35.7575 28.643)
+		(width 0.2)
+		(layer "B.Cu")
+		(net 77)
+	)
+	(segment

Commit message: Fix/exclude DRC errors
Parts:
- moved JP24 0.13 mm to (39.1, 57.5)
Connections:
- J4 pad 1: Net-(J4-Pin_1) -> /ET
- J4 pad 2: Net-(J4-Pin_2) -> /DT
- J4 pad 3: Net-(J4-Pin_3) -> /CT
- J4 pad 4: Net-(J4-Pin_4) -> /BT
- J4 pad 5: Net-(J4-Pin_5) -> /AT
- J5 pad 1: Net-(J5-Pin_1) -> /AB
- J5 pad 2: Net-(J5-Pin_2) -> /BB
- J5 pad 3: Net-(J5-Pin_3) -> /CB
- J5 pad 4: Net-(J5-Pin_4) -> /DB
- J5 pad 5: Net-(J5-Pin_5) -> /EB
- JP10 pad 1: Net-(J5-Pin_4) -> /DB
- JP11 pad 2: Net-(J4-Pin_1) -> /ET
- JP12 pad 1: Net-(J5-Pin_5) -> /EB
- JP15 pad 2: /A -> /AT
- JP16 pad 2: /B -> /BT
- JP17 pad 2: /C -> /CT
- JP18 pad 2: /D -> /DT
- JP19 pad 2: /E -> /ET
- JP20 pad 2: /A -> /AB
- JP21 pad 2: /B -> /BB
- JP22 pad 2: /C -> /CB
- JP23 pad 2: /D -> /DB
- JP24 pad 2: /E -> /EB
- JP3 pad 2: Net-(J4-Pin_5) -> /AT
- JP4 pad 1: Net-(J5-Pin_1) -> /AB
- JP5 pad 2: Net-(J4-Pin_4) -> /BT
- JP6 pad 1: Net-(J5-Pin_2) -> /BB
- JP7 pad 2: Net-(J4-Pin_3) -> /CT
- JP8 pad 1: Net-(J5-Pin_3) -> /CB
- JP9 pad 2: Net-(J4-Pin_2) -> /DT
Routing:
- net Net-(J22-Pin_23): track 0.11 -> 1.24 mm
Changed lines of the file:
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@@
 	(net 1 "VCC")
 	(net 2 "Net-(J2-Pin_1)")
-	(net 3 "Net-(J5-Pin_3)")
-	(net 4 "Net-(J5-Pin_5)")
+	(net 3 "/AT")
+	(net 4 "/BT")
 	(net 5 "Net-(J3-Pin_1)")
-	(net 6 "Net-(J5-Pin_4)")
-	(net 7 "Net-(J5-Pin_2)")
-	(net 8 "Net-(J4-Pin_3)")
-	(net 9 "Net-(J4-Pin_5)")
-	(net 10 "Net-(J4-Pin_4)")
-	(net 11 "Net-(J4-Pin_2)")
-	(net 12 "Net-(J4-Pin_1)")
-	(net 13 "Net-(J5-Pin_1)")
+	(net 6 "/ET")
+	(net 7 "/CT")
+	(net 8 "/DT")
+	(net 9 "/CB")
+	(net 10 "/EB")
+	(net 11 "/DB")
+	(net 12 "/BB")
+	(net 13 "/AB")
 	(net 14 "GND")
 	(net 15 "/8")
@@
 			(size 0.63 0.37)
 			(layers "F.Cu" "F.Mask")
-			(net 44 "/D")
+			(net 11 "/DB")
 			(pinfunction "B")
 			(pintype "passive")
@@
 			(size 0.63 0.37)
 			(layers "F.Cu" "F.Mask")
-			(net 43 "/C")
+			(net 9 "/CB")
 			(pinfunction "B")
 			(pintype "passive")
@@
 	(footprint "SMD:SolderJumper-2_0402_Bridged_Unmarked"
 		(layer "F.Cu")
-		(at 39.116 57.658 -135)
+		(at 39.091995 57.529605 -135)
 		(descr "SMD Solder Jumper, 0402 footprint, 0.3mm gap, bridged with 1 copper strip")
 		(tags "net tie solder jumper bridged")
@@
 			(size 0.63 0.37)
 			(layers "F.Cu" "F.Mask")
-			(net 45 "/E")
+			(net 10 "/EB")
 			(pinfunction "B")
 			(pintype "passive")
@@
 			(size 0.63 0.37)
 			(layers "F.Cu" "F.Mask")
-			(net 44 "/D")
+			(net 8 "/DT")
 			(pinfunction "B")
 			(pintype "passive")
@@
 			(size 0.63 0.37)
 			(layers "F.Cu" "F.Mask")
-			(net 41 "/A")
+			(net 3 "/AT")
 			(pinfunction "B")
 			(pintype "passive")
@@
 			(size 0.63 0.37)
 			(layers "F.Cu" "F.Mask")
-			(net 42 "/B")
+			(net 12 "/BB")
 			(pinfunction "B")
 			(pintype "passive")
@@
 			(size 0.63 0.37)
 			(layers "F.Cu" "F.Mask")
-			(net 41 "/A")
+			(net 13 "/AB")
 			(pinfunction "B")
 			(pintype "passive")
@@
 			(size 0.63 0.37)
 			(layers "F.Cu" "F.Mask")
-			(net 45 "/E")
+			(net 6 "/ET")
 			(pinfunction "B")
 			(pintype "passive")
@@
 			(size 0.63 0.37)
 			(layers "F.Cu" "F.Mask")
-			(net 42 "/B")
+			(net 4 "/BT")
 			(pinfunction "B")
 			(pintype "passive")
@@
 			(size 0.63 0.37)
 			(layers "F.Cu" "F.Mask")
-			(net 43 "/C")
+			(net 7 "/CT")
 			(pinfunction "B")
 			(pintype "passive")
@@
 			(size 0.63 0.37)
 			(layers "B.Cu" "B.Mask")
-			(net 6 "Net-(J5-Pin_4)")
+			(net 11 "/DB")
 			(pinfunction "A")
 			(pintype "passive")
@@
 			(size 0.63 0.37)
 			(layers "B.Cu" "B.Mask")
-			(net 13 "Net-(J5-Pin_1)")
+			(net 13 "/AB")
 			(pinfunction "A")
 			(pintype "passive")
@@
 			(size 0.63 0.37)
 			(layers "B.Cu" "B.Mask")
-			(net 10 "Net-(J4-Pin_4)")
+			(net 4 "/BT")
 			(pinfunction "B")
 			(pintype "passive")
@@
 			(size 0.63 0.37)
 			(layers "B.Cu" "B.Mask")
-			(net 11 "Net-(J4-Pin_2)")
+			(net 8 "/DT")
 			(pinfunction "B")
 			(pintype "passive")
@@
 			(remove_unused_layers no)
 			(roundrect_rratio 0.5)
-			(net 13 "Net-(J5-Pin_1)")
+			(net 13 "/AB")
 			(pinfunction "Pin_1")
 			(pintype "passive")
@@
 			(remove_unused_layers no)
 			(roundrect_rratio 0.5)
-			(net 13 "Net-(J5-Pin_1)")
+			(net 13 "/AB")
 			(pinfunction "Pin_1")
 			(pintype "passive")
@@
 			(remove_unused_layers no)
 			(roundrect_rratio 0.5)
-			(net 7 "Net-(J5-Pin_2)")
+			(net 12 "/BB")
 			(pinfunction "Pin_2")
 			(pintype "passive")
@@
 			(remove_unused_layers no)
 			(roundrect_rratio 0.5)
-			(net 7 "Net-(J5-Pin_2)")
+			(net 12 "/BB")
 			(pinfunction "Pin_2")
 			(pintype "passive")
@@
 			(remove_unused_layers no)
 			(roundrect_rratio 0.5)
-			(net 3 "Net-(J5-Pin_3)")
+			(net 9 "/CB")
 			(pinfunction "Pin_3")
 			(pintype "passive")
@@
 			(remove_unused_layers no)
 			(roundrect_rratio 0.5)
-			(net 3 "Net-(J5-Pin_3)")
+			(net 9 "/CB")
 			(pinfunction "Pin_3")
 			(pintype "passive")
@@
 			(remove_unused_layers no)
 			(roundrect_rratio 0.5)
-			(net 6 "Net-(J5-Pin_4)")
+			(net 11 "/DB")
 			(pinfunction "Pin_4")
 			(pintype "passive")
@@
 			(remove_unused_layers no)
 			(roundrect_rratio 0.5)
-			(net 6 "Net-(J5-Pin_4)")
+			(net 11 "/DB")
 			(pinfunction "Pin_4")
 			(pintype "passive")
@@
 			(remove_unused_layers no)
 			(roundrect_rratio 0.5)
-			(net 4 "Net-(J5-Pin_5)")
+			(net 10 "/EB")
 			(pinfunction "Pin_5")
 			(pintype "passive")
@@
 			(remove_unused_layers no)
 			(roundrect_rratio 0.5)
-			(net 4 "Net-(J5-Pin_5)")
+			(net 10 "/EB")
 			(pinfunction "Pin_5")
 			(pintype "passive")
@@
 			(size 0.63 0.37)
 			(layers "B.Cu" "B.Mask")
-			(net 7 "Net-(J5-Pin_2)")
+			(net 12 "/BB")
 			(pinfunction "A")
 			(pintype "passive")
@@
 			(size 0.63 0.37)
 			(layers "B.Cu" "B.Mask")
-			(net 8 "Net-(J4-Pin_3)")
+			(net 7 "/CT")
 			(pinfunction "B")
 			(pintype "passive")
@@
 			(size 0.63 0.37)
 			(layers "B.Cu" "B.Mask")
-			(net 3 "Net-(J5-Pin_3)")
+			(net 9 "/CB")
 			(pinfunction "A")
 			(pintype "passive")
@@
 			(size 0.63 0.37)
 			(layers "B.Cu" "B.Mask")
-			(net 9 "Net-(J4-Pin_5)")
+			(net 3 "/AT")
 			(pinfunction "B")
 			(pintype "passive")
@@
 			(size 0.63 0.37)
 			(layers "B.Cu" "B.Mask")
-			(net 4 "Net-(J5-Pin_5)")
+			(net 10 "/EB")
 			(pinfunction "A")
 			(pintype "passive")
@@
 			(remove_unused_layers no)
 			(roundrect_rratio 0.5)
-			(net 12 "Net-(J4-Pin_1)")
+			(net 6 "/ET")
 			(pinfunction "Pin_1")
 			(pintype "passive")
@@
 			(remove_unused_layers no)
 			(roundrect_rratio 0.5)
-			(net 12 "Net-(J4-Pin_1)")
+			(net 6 "/ET")
 			(pinfunction "Pin_1")
 			(pintype "passive")
@@
 			(remove_unused_layers no)
 			(roundrect_rratio 0.5)
-			(net 11 "Net-(J4-Pin_2)")
+			(net 8 "/DT")
 			(pinfunction "Pin_2")
 			(pintype "passive")
@@
 			(remove_unused_layers no)
 			(roundrect_rratio 0.5)
-			(net 11 "Net-(J4-Pin_2)")
+			(net 8 "/DT")
 			(pinfunction "Pin_2")
 			(pintype "passive")
@@
 			(remove_unused_layers no)
 			(roundrect_rratio 0.5)
-			(net 8 "Net-(J4-Pin_3)")
+			(net 7 "/CT")
 			(pinfunction "Pin_3")
 			(pintype "passive")
@@
 			(remove_unused_layers no)
 			(roundrect_rratio 0.5)
-			(net 8 "Net-(J4-Pin_3)")
+			(net 7 "/CT")
 			(pinfunction "Pin_3")
 			(pintype "passive")
@@
 			(remove_unused_layers no)
 			(roundrect_rratio 0.5)
-			(net 10 "Net-(J4-Pin_4)")
+			(net 4 "/BT")
 			(pinfunction "Pin_4")
 			(pintype "passive")
@@
 			(remove_unused_layers no)
 			(roundrect_rratio 0.5)
-			(net 10 "Net-(J4-Pin_4)")
+			(net 4 "/BT")
 			(pinfunction "Pin_4")
 			(pintype "passive")
@@
 			(remove_unused_layers no)
 			(roundrect_rratio 0.5)
-			(net 9 "Net-(J4-Pin_5)")
+			(net 3 "/AT")
 			(pinfunction "Pin_5")
 			(pintype "passive")
@@
 			(remove_unused_layers no)
 			(roundrect_rratio 0.5)
-			(net 9 "Net-(J4-Pin_5)")
+			(net 3 "/AT")
 			(pinfunction "Pin_5")
 			(pintype "passive")
@@
 			(size 0.63 0.37)
 			(layers "B.Cu" "B.Mask")
-			(net 12 "Net-(J4-Pin_1)")
+			(net 6 "/ET")
 			(pinfunction "B")
 			(pintype "passive")
@@
 	)
 	(segment
+		(start 38.03875 28.6487)
+		(end 38.03875 29.7713)
+		(width 0.2)
+		(layer "F.Cu")
+		(net 79)
+	)
+	(segment
